Commit message: commit

File: urdf/mbot.xacro (robot description, xacro)
@@ -1,12 +1,12 @@
 <?xml version="1.0"?>
 <robot name="mbot" xmlns:xacro="http://www.ros.org/wiki/xacro">
-	<!--<xacro:include filename="$(find mbot_pointer)/urdf/mbot.gazebo"/>-->
-	<xacro:include filename="$(find mbot_pointer)/urdf/materials.xacro"/>
-	<link name = "base_link">
+	<link name ="base_link">
 		<visual>
 			<geometry>
 				<box size = "0.2 0.1 0.1"/>
 			</geometry>
-			<material name ="blue"/>
+			<material name ="blue">
+				<color rgba="0.0 0.0 0.8 1.0"/>
+			</material>
 		</visual>
 		<collision>
@@ -19,12 +19,12 @@
 			<inertia ixx="0.00667" ixy="0.0" ixz="0.0" iyy="0.00667" iyz="0.0" izz="0.00267"/>
 		</inertial>
-		<gazebo reference="base_link">
-        	<!--<mu1 value="200.0"/>-->
-        	<!--<mu2 value="100.0"/>-->
-        	<!--<kp value="10000000.0" />-->
-        	<!--<kd value="1.0" />-->
-        	<material>Gazebo/Blue</material>
-    	</gazebo>
 	</link>
+	<gazebo reference="base_link">
+		<!--<mu1 value="200.0"/>-->
+		<!--<mu2 value="100.0"/>-->
+		<!--<kp value="10000000.0" />-->
+		<!--<kd value="1.0" />-->
+		<material>Gazebo/Blue</material>
+	</gazebo>
 	<xacro:macro name="wheel_tran" params="prefix suffix">
 		<transmission name="tran_${prefix}_${suffix}">
@@ -45,5 +45,7 @@
 				</geometry>
 				<origin rpy="1.57075 0 0" xyz="0 0 0"/>
-				<material name="black"/>
+				<material name="black">
+					<color rgba="0.0 0.0 0.0 1.0"/>
+				</material>
 			</visual>
 			<collision>
@@ -77,44 +79,118 @@
 	<xacro:wheel_link prefix="rear" suffix="left" xreflect="-1.0" yreflect="1.0"/>
 	<xacro:wheel_link prefix="rear" suffix="right" xreflect="-1.0" yreflect="-1.0"/>
-    <link name="imu">
+    <link name="imu_link">
         <visual>
             <geometry>
                 <box size="0.001 0.001 0.0001"/>
             </geometry>
-            <material name="grey"/>
+            <material name="grey">
+				<color rgba="0.2 0.2 0.2 1.0"/>
+			</material>
         </visual>
+		<collision>
+			<geometry>
+                <box size="0.001 0.001 0.0001"/>
+            </geometry>
+		</collision>
 		<inertial>
 			<mass value="0.01"/>
 			<inertia ixx="0.000001" ixy="0.0" ixz="0.0" iyy="0.000001" iyz="0.0" izz="0.0000001"/>
 		</inertial>
-		<gazebo reference="imu">
-			<material>Gazebo/Grey</material>
-		</gazebo>
     </link>
-    <joint name="base_ot_imu" type="fixed">
+    <joint name="base_to_imu" type="fixed">
+		<axis rpy="0 0 0" xyz="0 0 1"/>
         <parent link="base_link"/>
-        <child link="imu"/>
+        <child link="imu_link"/>
         <origin rpy="0 0 0" xyz="0 0 0.05"/>
     </joint>
-    <link name="xtion">
+	<gazebo reference="imu_link">
+		<gravity>true</gravity>
+		<material>Gazebo/Grey</material>
+		<sensor name="imu_sensor" type="imu">
+			<always_on>true</always_on>
+			<update_rate>100</update_rate>
+			<visualize>true</visualize>
+			<topic>imu</topic>
+			<plugin filename="libgazebo_ros_imu_sensor.so" name="imu_plugin">
+				<topicName>imu</topicName>
+				<bodyName>imu</bodyName>
+				<updateRateHZ>10.0</updateRateHZ>
+				<gaussianNoise>0.0</gaussianNoise>
+				<xyzOffset>0 0 0</xyzOffset>
+				<rpyOffset>0 0 0</rpyOffset>
+				<frameName>imu</frameName>
+			</plugin>
+			<pose>0 0 0 0 0 0</pose>
+		</sensor>
+	</gazebo>
+    <link name="xtion_link">
         <visual>
             <geometry>
                 <box size="0.05 0.18 0.03"/>
             </geometry>
-            <material name="green"/>
+			<material name="green">
+				<color rgba="0.0 0.8 0.0 1.0"/>
+			</material>
         </visual>
+		<collision>
+			<geometry>
+                <box size="0.05 0.18 0.03"/>
+            </geometry>
+		</collision>
 		<inertial>
 			<mass value="0.1"/>
 			<inertia ixx="0.0000283" ixy="0.0" ixz="0.0" iyy="0.0002775" iyz="0.0" izz="0.00029"/>
 		</inertial>
-		<gazebo reference="xtion">
-			<material>Gazebo/Green</material>
-		</gazebo>
     </link>
     <joint name="base_to_xtion" type="fixed">
+		<axis rpy="0 0 0" xyz="0 0 1"/>
         <parent link="base_link"/>
-        <child link="xtion"/>
+        <child link="xtion_link"/>
         <origin rpy="0 0 0" xyz="0.068 0 0.065"/>
     </joint>
+	<gazebo reference="xtion_link">
+		<material>Gazebo/Green</material>
+		<sensor type="depth" name="xtion">
+			<pose>0 0 0 0 0 0</pose>
+			<always_on>true</always_on>
+			<visualize>true</visualize>
+			<camera>
+				<horizontal_fov>1.02974</horizontal_fov>
+				<image>
+					<width>640</width>
+					<height>480</height>
+					<format>R8G8B8</format>
+				</image>
+				<depth_camera></depth_camera>
+				<clip>
+					<near>0.02</near>
+					<far>300</far>
+				</clip>
+			</camera>
+			<plugin name="$xtion_link_controller" filename="libgazebo_ros_openni_kinect.so">
+				<baseline>0.2</baseline>
+				<alwaysOn>true</alwaysOn>
+				<updateRate>30.0</updateRate>
+				<cameraName>camera</cameraName>
+				<imageTopicName>/camera/rgb/image_raw</imageTopicName>
+				<cameraInfoTopicName>/camera/rgb/camera_info</cameraInfoTopicName>
+				<depthImageTopicName>/camera/depth/image_raw</depthImageTopicName>
+				<depthImageInfoTopicName>/camera/depth/camera_info</depthImageInfoTopicName>
+				<pointCloudTopicName>/camera/depth/points</pointCloudTopicName>
+				<frameName>xtion_link</frameName>
+				<pointCloudCutoff>0.5</pointCloudCutoff>
+				<distortionK1>0.00000001</distortionK1>
+				<distortionK2>0.00000001</distortionK2>
+				<distortionK3>0.00000001</distortionK3>
+				<distortionT1>0.00000001</distortionT1>
+				<distortionT2>0.00000001</distortionT2>
+				<CxPrime>0</CxPrime>
+				<Cx>0</Cx>
+				<Cy>0</Cy>
+				<focalLength>0</focalLength>
+				<hackBaseline>0</hackBaseline>
+			</plugin>
+		</sensor>
+	</gazebo>
 	<gazebo>
         <plugin name="gazebo_ros_control" filename="libgazebo_ros_control.so">
